File: AXAWIFI.brd (EAGLE design)
At the start: 94 x 27.9 mm, 25 parts, among them IC1 MCP2003, IC2 ESP12SMT, SW1 RESET, SW2 REFLASH

Commit message: Replaced parts using SuperHouse library
Parts:
- removed C2: 10uF 6.3V A TANT, freetronics:EIA3216
- removed IC2: ESP12SMT, freetronics-jon:ESP12
- added C5: 10uF, SuperHouse-DiscreteSemi:C0805
- added U$1: ESP12-SMT, SuperHouse-MCUs:ESP12
- C4: device freetronics-jon:0603 -> SuperHouse-DiscreteSemi:C0603
- JP3: value (none) -> M06-PIN; device freetronics-master-v1:1X06 -> SuperHouse-Connectors:1X06-P
- JP4: device freetronics-master-v1.1:SCREWTERMINAL-3.5MM-2 -> SuperHouse-Connectors:SCREWTERMINAL-3.5MM-2
- LED1, LED2: device freetronics-jon:LED-0603 -> SuperHouse-LEDs:LED-0603
- R10, R11, R12, R2, R3, R4, R5, R6, R7, R8, R9: device freetronics-jon:0603 -> SuperHouse-DiscreteSemi:R0603
- REG1: device freetronics-jon:K78XX-500R3 -> SuperHouse-Regulators:K78XX-500R3
- SW1, SW2: device freetronics-jon:TACTILE_SWITCH_SMD_2PIN_TINY -> SuperHouse-Switches:TACTILE_SMT_3X4X2
Connections:
- net 3.3V: now also C5.1, U$1.8; no longer C2.A, IC2.8
- net ADC: now also U$1.2; no longer IC2.2
- net CH_PD: now also U$1.3; no longer IC2.3
- net GND: now also C5.2, U$1.9; no longer C2.C, IC2.9
- net GPIO0: now also U$1.12; no longer IC2.12
- net GPIO12: now also U$1.6; no longer IC2.6
- net GPIO13: now also U$1.7; no longer IC2.7
- net GPIO14: now also U$1.5; no longer IC2.5
- net GPIO15: now also U$1.10; no longer IC2.10
- net GPIO16: now also U$1.4; no longer IC2.4
- net GPIO2: now also U$1.11; no longer IC2.11
- net GPIO4: now also U$1.14; no longer IC2.14
- net GPIO5: now also U$1.13; no longer IC2.13
- net RST: now also U$1.1; no longer IC2.1
- net RX: now also U$1.15; no longer IC2.15
- net TX: now also U$1.16; no longer IC2.16

Commit message: Replaced programming header with ESProg header
Parts:
- removed JP3: M06-PIN, SuperHouse-Connectors:1X06-P
- added J1: ESPROG-SOCKET, SuperHouse-Connectors:ESPROG-S
- moved R6 1.27 mm to (54.7, 21.0)
Connections:
- removed net RST: R3.1, SW1.1, U$1.1
- new net !RST: J1.6, R3.1, SW1.1, U$1.1
- net 3.3V: now also J1.3; no longer JP3.3
- net GND: now also J1.1; no longer JP3.1
- net GPIO0: now also J1.2
- net RX: now also J1.4; no longer JP3.4
- net TX: now also J1.5; no longer JP3.5
Routing:
- net !RST: track 0.00 -> 30.5 mm, vias 0 -> 1
- net RST: track 15.2 -> 0.00 mm
- net TX: track 80.4 -> 69.2 mm
- net 3.3V: track 152.2 -> 146.2 mm
- net GPIO0: track 79.3 -> 84.3 mm
- net RX: track 63.4 -> 64.5 mm
- added copper zone on layer 16, net 3.3V
- removed copper zone on layer 16, net GND
Other:
- board text added: "ESProg"
- board text removed: "3.3V FTDI"
- board text removed: "BLK"
- board text removed: "GRN"

Commit message: Replace parts using SuperHouse library for 3D models
Parts:
- C1, C3: device analyzer:UD-6,3X5,8_NICHICON -> SuperHouse-DiscreteSemi:PANASONIC_C
- IC1: device freetronics-jon:SOIC8T -> SuperHouse-ICs:SOIC8T
- JP2: device freetronics-jon:1X03 -> SuperHouse-Connectors:1X03
- moved JP4 1.27 mm to (11.1, 5.08)
Connections:
- net +12V renamed 12V
Routing:
- net 3.3V: track 146.2 -> 145.7 mm
